Commit message: changing stupidbot build urdf organization

File: src/stupidbot/stupidbot/stupidbot_description/robot/stupidbot.urdf.xacro (robot description, xacro)
@@ -1,6 +1,48 @@
 <?xml version="1.0"?>
-<robot name="stupidbot" xmlns:xacro="http://ros.org/wiki/xacro">
+<robot name="stupidbot" xmlns:xacro="http://www.ros.org/wiki/xacro">
 	<xacro:include filename="$(find stupidbot_description)/urdf/stupidbot_library.urdf.xacro"/>
-	<stupidbot_chassis/>
+	<material name="black">
+		<color rgba="0 0 0 1"/>
+	</material>
+	<!-- Base link, center of chassis and body -->
+	<link name="base_link">
+		<visual>
+			<geometry>
+				<box size="${chassis_length} ${chassis_width} ${chassis_height}"/>
+			</geometry>
+		</visual>
+		<inertial>
+			<mass value="20"/>
+			<inertia ixx="${chassis_mass*(chassis_length*chassis_length + chassis_height*chassis_height)/12}" ixy="0.0" ixz="0.0" iyy="${chassis_mass*(chassis_width*chassis_width + chassis_height*chassis_height)/12}" iyz="0.0" izz="${chassis_mass*(chassis_length*chassis_length + chassis_width*chassis_width)/12}"/>
+		</inertial>
+		<collision>
+			<geometry>
+				<box size="${chassis_length} ${chassis_width} ${chassis_height}"/>
+			</geometry>
+			<origin xyz="0 0 0" rpy="0 0 0"/>
+		</collision>
+		<gazebo reference="base_link"/>
+	</link>
+	<link name="base_footprint">
+		<visual>
+			<geometry>
+				<box size="0.001 0.001 0.001"/>
+			</geometry>
+			<origin xyz="0 0 0" rpy="0 0 0"/>
+		</visual>
+		<inertial>
+			<mass value="0.0001"/>
+			<origin xyz="0 0 0"/>
+			<inertia ixx="0.0001" ixy="0.0" ixz="0.0" iyy="0.0001" iyz="0.0" izz="0.0001"/>
+		</inertial>
+	</link>
+	<joint name="base_footprint_joint" type="fixed">
+		<origin xyz="0 0 0.06"/>
+		<parent link="base_footprint"/>
+		<child link="base_link"/>
+	</joint>
+	<wheel lr="right" parent="base_link" reflectY="1" />
+	<wheel lr="left" parent="base_link" reflectY="-1" />
+	<caster parent="base_link" fb="front" reflectX="1"/>
 	<differential_skid/>
 </robot>

File: src/stupidbot/stupidbot/stupidbot_description/urdf/stupidbot_gazebo.urdf.xacro (robot description, xacro)
@@ -8,15 +8,18 @@
 				<alwaysOn>true</alwaysOn>
 				<updateRate>100.0</updateRate>
-				<robotNamespace>/</robotNamespace>
-				<leftJoint>base_to_left_wheel</leftJoint>
-				<rightJoint>base_to_right_wheel</rightJoint>
+				<leftJoint>left_wheel_joint</leftJoint>
+				<rightJoint>right_wheel_joint</rightJoint>
+				<wheelSeparation>${chassis_width + 0.02}</wheelSeparation>
+				<wheelDiameter>0.12</wheelDiameter>
+				<wheelTorque>10</wheelTorque>
+				<robotBaseFrame>base_footprint</robotBaseFrame>
+				<odometryFrame>map</odometryFrame>
+				<publishWheelJointState>true</publishWheelJointState>
 				<publishWheelTF>true</publishWheelTF>
-				<publishWheelJointState>true</publishWheelJointState>
-				<publishTF>1</publishTF>
-				<wheelSeparation>${chassis_width}</wheelSeparation>
-				<wheelDiameter>${2*wheel_radius}</wheelDiameter>
-				<robotBaseFrame>base_link</robotBaseFrame>
 			</plugin>
 			<plugin name="gazebo_ros_control" filename="libgazebo_ros_control.so"/>
+			<plugin name="gazebo_ros_joint_state_publisher" filename="libgazebo_ros_joint_state_publisher.so">
+				<jointName>front_caster_swivel_joint, front_caster_joint</jointName>
+			</plugin>
 		</gazebo>
 	</xacro:macro>

File: src/stupidbot/stupidbot/stupidbot_description/urdf/stupidbot_library.urdf.xacro (robot description, xacro)
@@ -3,6 +3,8 @@
 	<!-- General robot properties -->
 	<xacro:include filename="$(find stupidbot_description)/urdf/stupidbot_properties.urdf.xacro"/>
-	<!-- Robot body creation macros -->
-	<xacro:include filename="$(find stupidbot_description)/urdf/stupidbot_chassis.urdf.xacro"/>
+	<!-- Robot wheel creation macro -->
+	<xacro:include filename="$(find stupidbot_description)/urdf/stupidbot_wheel.urdf.xacro"/>
+	<!-- Caster wheel macro -->
+	<xacro:include filename="$(find stupidbot_description)/urdf/stupidbot_caster.urdf.xacro"/>
 	<!-- Gazebo descriptions -->
 	<xacro:include filename="$(find stupidbot_description)/urdf/stupidbot_gazebo.urdf.xacro"/>

File: src/stupidbot/stupidbot/stupidbot_description/urdf/stupidbot_properties.urdf.xacro (robot description, xacro)
@@ -4,7 +4,4 @@
 	<property name="chassis_width" value="0.2"/>
 	<property name="chassis_height" value="0.05"/>
-	<property name="wheel_width" value="0.04"/>
-	<property name="wheel_radius" value="0.06"/>
-	<property name="caster_width" value="0.02"/>
-	<property name="caster_radius" value="0.02"/>
+	<property name="chassis_mass" value="20.0"/>
 </robot>

Commit message: added camera, put most description values in properties

File: src/stupidbot/stupidbot/stupidbot_description/robot/stupidbot.urdf.xacro (robot description, xacro)
@@ -14,5 +14,5 @@
 		<inertial>
 			<mass value="20"/>
-			<inertia ixx="${chassis_mass*(chassis_length*chassis_length + chassis_height*chassis_height)/12}" ixy="0.0" ixz="0.0" iyy="${chassis_mass*(chassis_width*chassis_width + chassis_height*chassis_height)/12}" iyz="0.0" izz="${chassis_mass*(chassis_length*chassis_length + chassis_width*chassis_width)/12}"/>
+			<inertia ixx="${chassis_ixx}" ixy="0.0" ixz="0.0" iyy="${chassis_iyy}" iyz="0.0" izz="${chassis_izz}"/>
 		</inertial>
 		<collision>
@@ -24,4 +24,5 @@
 		<gazebo reference="base_link"/>
 	</link>
+	<!-- Base footprint as a reference to the ground beneath robot -->
 	<link name="base_footprint">
 		<visual>
@@ -36,13 +37,23 @@
 			<inertia ixx="0.0001" ixy="0.0" ixz="0.0" iyy="0.0001" iyz="0.0" izz="0.0001"/>
 		</inertial>
+		<gazebo reference="base_footprint"/>
 	</link>
+	<!-- Joint connecting base_link to the footprint -->
 	<joint name="base_footprint_joint" type="fixed">
 		<origin xyz="0 0 0.06"/>
 		<parent link="base_footprint"/>
 		<child link="base_link"/>
+		<gazebo reference="base_footprint_joint"/>
 	</joint>
+	<!-- Wheels, complete specification including links and joints -->
 	<wheel lr="right" parent="base_link" reflectY="1" />
 	<wheel lr="left" parent="base_link" reflectY="-1" />
-	<caster parent="base_link" fb="front" reflectX="1"/>
-	<differential_skid/>
+	<!-- Caster(s), complete specification including links and joints -->
+	<caster parent="base_link" lr="right" reflectY="-1"/>
+	<caster parent="base_link" lr="left" reflectY="1"/>
+	<!-- Camera -->
+	<stupidbot_camera parent="base_link"/>
+	<!-- Start gazebo plugins, diff_drive and joint state publisher as of now -->
+	<stupidbot_gazebo/>
+	<gazebo reference="stupidbot"/>
 </robot>

File: src/stupidbot/stupidbot/stupidbot_description/urdf/stupidbot_caster.urdf.xacro (robot description, xacro)
@@ -1,15 +1,10 @@
 <?xml version="1.0"?>
 <robot xmlns:xacro="http://www.ros.org/wiki/xacro">
+	<!-- Properties file -->
 	<xacro:include filename="$(find stupidbot_description)/urdf/stupidbot_properties.urdf.xacro"/>
-	<!-- Caster constant properties -->
-	<xacro:property name="caster_width" value="0.015"/>
-	<xacro:property name="caster_radius" value="0.016"/>
-	<xacro:property name="caster_mass" value="8.0"/>
-	<xacro:property name="caster_ixx" value="${caster_mass*(3*caster_radius*caster_radius + caster_width*caster_width)/12}"/>
-	<xacro:property name="caster_iyy" value="${caster_mass*(caster_radius*caster_radius)/2}"/>
-	<xacro:property name="caster_izz" value="${caster_mass*(3*caster_radius*caster_radius + caster_width*caster_width)/12}"/>
-	<xacro:macro name="caster" params="parent fb reflectX">
+	<!-- Full caster description including swivel and wheel -->
+	<xacro:macro name="caster" params="parent lr reflectY">
 		<!-- Caster swivel -->
-		<link name="${fb}_caster_swivel">
+		<link name="${lr}_caster_swivel">
 			<visual>
 				<geometry>
@@ -27,8 +22,8 @@
 				</geometry>
 			</collision>
-			<gazebo reference="${fb}_caster_swivel"/>
+			<gazebo reference="${lr}_caster_swivel"/>
 		</link>
 		<!-- Caster wheel -->
-		<link name="${fb}_caster_wheel">
+		<link name="${lr}_caster_wheel">
 			<visual>
 				<geometry>
@@ -48,30 +43,31 @@
 				<origin rpy="1.57057 0 0"/>
 			</collision>
-			<gazebo reference="${fb}_caster_wheel">
-				<mu1 value="0.0"/>
-				<mu2 value="0.0"/>
-				<kp value="1000000.0"/>
-				<kd value="100.0"/>
-			</gazebo>
 		</link>
+		<!-- Set Gazebo physics parameters -->
+		<gazebo reference="${lr}_caster_wheel">
+			<mu1>0.7</mu1>
+			<mu2>0.7</mu2>
+			<kp>10000000</kp>
+			<kd>100.0</kd>
+			<minDepth>0.001</minDepth>
+		</gazebo>
 		<!-- Joint connecting base and caster swivel -->
-		<joint name="${fb}_caster_swivel_joint" type="revolute">
+		<joint name="${lr}_caster_swivel_joint" type="revolute">
 			<parent link="${parent}"/>
-			<child link="${fb}_caster_swivel"/>
+			<child link="${lr}_caster_swivel"/>
 			<axis xyz="0 0 1"/>
-			<origin xyz="${reflectX*chassis_length/4} 0 -${chassis_height/2 + 0.005}"/>
-			<limit upper="1.57057" lower="-1.57057" effort="100.0" velocity="0.0"/>
-			<gazebo reference="${fb}_caster_swivel_joint"/>
+			<origin xyz="${chassis_length/4} ${reflectY * caster_y_displacement} -${chassis_height/2 + 0.005}"/>
+			<limit upper="3.1415" lower="-3.1415" effort="100.0" velocity="0.0"/>
 		</joint>
+		<gazebo reference="${lr}_caster_swivel_joint"/>
 		<!-- Joint connecting caster swivel and caster -->
-		<joint name="${fb}_caster_joint" type="continuous">
-			<parent link="${fb}_caster_swivel"/>
-			<child link="${fb}_caster_wheel"/>
+		<joint name="${lr}_caster_joint" type="continuous">
+			<parent link="${lr}_caster_swivel"/>
+			<child link="${lr}_caster_wheel"/>
 			<axis xyz="0 1 0"/>
 			<origin xyz="0 0 -${caster_radius + 0.003}"/>
 			<limit effort="100.0" velocity="0.0"/>
-			<dynamics damping="1.0"/>
-			<gazebo reference="${fb}_caster_joint"/>
 		</joint>
+		<gazebo reference="${lr}_caster_joint"/>
 	</xacro:macro>
 </robot>

File: src/stupidbot/stupidbot/stupidbot_description/urdf/stupidbot_gazebo.urdf.xacro (robot description, xacro)
@@ -1,8 +1,10 @@
 <?xml version="1.0"?>
 <robot name="stupidbot_gazebo" xmlns:xacro="http://www.ros.org/wiki/xacro">
-	<!-- Differential Drive -->
-	<xacro:macro name="differential_skid">
+	<!-- Set up for all model plugins -->
+	<xacro:macro name="stupidbot_gazebo">
+	<!-- Include properties file -->
 	<xacro:include filename="$(find stupidbot_description)/urdf/stupidbot_properties.urdf.xacro"/>
 		<gazebo>
+			<!-- Differential Drive Plugin -->
 			<plugin name="diff_drive_controller" filename="libgazebo_ros_diff_drive.so">
 				<alwaysOn>true</alwaysOn>
@@ -18,7 +20,10 @@
 				<publishWheelTF>true</publishWheelTF>
 			</plugin>
+			<!-- Ros Control Plugin -->
 			<plugin name="gazebo_ros_control" filename="libgazebo_ros_control.so"/>
+			<!-- Joint State Publisher for non-actuated joints -->
+			<!-- Place any joints we want published in the jointName tag -->
 			<plugin name="gazebo_ros_joint_state_publisher" filename="libgazebo_ros_joint_state_publisher.so">
-				<jointName>front_caster_swivel_joint, front_caster_joint</jointName>
+				<jointName>left_caster_swivel_joint, left_caster_joint, right_caster_swivel_joint, right_caster_joint</jointName>
 			</plugin>
 		</gazebo>

File: src/stupidbot/stupidbot/stupidbot_description/urdf/stupidbot_library.urdf.xacro (robot description, xacro)
@@ -7,4 +7,6 @@
 	<!-- Caster wheel macro -->
 	<xacro:include filename="$(find stupidbot_description)/urdf/stupidbot_caster.urdf.xacro"/>
+	<!-- Camera macro -->
+	<xacro:include filename="$(find stupidbot_description)/urdf/sensors/stupidbot_camera.urdf.xacro"/>
 	<!-- Gazebo descriptions -->
 	<xacro:include filename="$(find stupidbot_description)/urdf/stupidbot_gazebo.urdf.xacro"/>

File: src/stupidbot/stupidbot/stupidbot_description/urdf/stupidbot_properties.urdf.xacro (robot description, xacro)
@@ -1,7 +1,37 @@
 <?xml version="1.0"?>
 <robot>
+	<!-- Chassis/body properties -->
 	<property name="chassis_length" value="0.2"/>
 	<property name="chassis_width" value="0.2"/>
 	<property name="chassis_height" value="0.05"/>
-	<property name="chassis_mass" value="20.0"/>
+	<property name="chassis_mass" value="40.0"/>
+	<property name="chassis_ixx" value="${chassis_mass*(chassis_length*chassis_length + chassis_height*chassis_height)/12}"/>
+	<property name="chassis_iyy" value="${chassis_mass*(chassis_width*chassis_width + chassis_height*chassis_height)/12}"/>
+	<property name="chassis_izz" value="${chassis_mass*(chassis_length*chassis_length + chassis_width*chassis_width)/12}"/>
+	<!-- Wheel properties -->
+	<property name="wheel_mass" value="10.0"/>
+	<property name="wheel_radius" value="0.06"/>
+	<property name="wheel_width" value="0.04"/>
+	<property name="wheel_ixx" value="${(wheel_mass*(3*wheel_radius*wheel_radius + wheel_width*wheel_width))/12}"/>
+	<property name="wheel_iyy" value="${(wheel_mass*(3*wheel_radius*wheel_radius + wheel_width*wheel_width))/12}"/>
+	<property name="wheel_izz" value="${(wheel_mass*wheel_radius*wheel_radius)/2}"/>
+	<!-- Camera properties -->
+	<property name="camera_mass" value="0.5"/>
+	<property name="camera_length" value="0.02"/>
+	<property name="camera_width" value="0.02"/>
+	<property name="camera_height" value="0.02"/>
+	<property name="camera_x_pos" value="${chassis_length/2 - camera_length/2}"/>
+	<property name="camera_y_pos" value="-${chassis_width/4}"/>
+	<property name="camera_z_pos" value="${chassis_height/2 + camera_height/2}"/>
+	<property name="camera_ixx" value="${camera_mass*(camera_length*camera_length + camera_height*camera_height)/12}"/>
+	<property name="camera_iyy" value="${camera_mass*(camera_width*camera_width + camera_height*camera_height)/12}"/>
+	<property name="camera_izz" value="${camera_mass*(camera_length*camera_length + camera_width*camera_width)/12}"/>
+	<!-- Caster properties -->
+	<property name="caster_width" value="0.015"/>
+	<property name="caster_radius" value="0.012"/>
+	<property name="caster_mass" value="5.0"/>
+	<property name="caster_ixx" value="${caster_mass*(3*caster_radius*caster_radius + caster_width*caster_width)/12}"/>
+	<property name="caster_iyy" value="${caster_mass*(3*caster_radius*caster_radius + caster_width*caster_width)/12}"/>
+	<property name="caster_izz" value="${caster_mass*(caster_radius*caster_radius)/2}"/>
+	<property name="caster_y_displacement" value="${chassis_width/4}"/>
 </robot>

File: src/stupidbot/stupidbot/stupidbot_description/urdf/stupidbot_wheel.urdf.xacro (robot description, xacro)
@@ -1,10 +1,7 @@
 <?xml version="1.0"?>
-<robot name="wheels" xmlns:xacro="http://www.ros.org/wiki/xacro">
+<robot xmlns:xacro="http://www.ros.org/wiki/xacro">
 	<!-- Include chassis properties for positioning joints -->
 	<xacro:include filename="$(find stupidbot_description)/urdf/stupidbot_properties.urdf.xacro"/>
-	<!-- Wheel properties -->
-	<xacro:property name="wheel_mass" value="10.0"/>
-	<xacro:property name="wheel_radius" value="0.06"/>
-	<xacro:property name="wheel_width" value="0.04"/>
+	<!-- Full description macro for wheel including transmissions, etc -->
 	<xacro:macro name="wheel" params="lr parent reflectY">
 		<!-- Wheel link description -->
@@ -19,5 +16,5 @@
 			<inertial>
 				<mass value="${wheel_mass}"/>
-				<inertia ixx="${(wheel_mass*(3*wheel_radius*wheel_radius + wheel_width*wheel_width))/12}" ixy="0.0" ixz="0.0" iyy="${(wheel_mass*(3*wheel_radius*wheel_radius + wheel_width*wheel_width))/12}" iyz="0.0" izz="${(wheel_mass*wheel_radius*wheel_radius)/2}"/>
+				<inertia ixx="${wheel_ixx}" ixy="0.0" ixz="0.0" iyy="${wheel_iyy}" iyz="0.0" izz="${wheel_izz}"/>
 			</inertial>
 			<collision>
@@ -27,11 +24,13 @@
 				<origin rpy="1.57057 0 0"/>
 			</collision>
-			<gazebo reference="${lr}_wheel">
-				<mu1 value="1.0"/>
-				<mu2 value="1.0"/>
-				<kp  value="10000000.0" />
-      			<kd  value="100.0" />
-			</gazebo>
 		</link>
+		<!-- Gazebo description for wheel -->
+		<gazebo reference="${lr}_wheel">
+			<mu1>1.0</mu1>
+			<mu2>1.0</mu2>
+			<kp>10000000.0</kp>
+			<kd>100.0</kd>
+			<minDepth>0.001</minDepth>
+		</gazebo>
 		<!-- Joint connecting wheel and base link -->
 		<joint name="${lr}_wheel_joint" type="continuous">
@@ -41,6 +40,7 @@
 			<origin xyz="-${chassis_length/4} ${reflectY * (chassis_width/2 + wheel_width/2)} 0"/>
 			<limit effort="100" velocity="0.0"/>
-			<gazebo reference="${lr}_wheel_joint"/>
 		</joint>
+		<!-- Gazebo description for wheel_joint -->
+		<gazebo reference="${lr}_wheel_joint"/>
 		<!-- Transmission for wheel joint -->
 		<transmission name="${lr}_wheel_trans">
